File: kicad_files/loki65.kicad_sch (KiCad schematic)
At the start: 214 parts, among them J1 TYPE-C-31-M-12, SW1 MX style mechanical keyboard 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, SW10 MX style mechanical keyboard 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, SW11 MX style mechanical keyboard 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, SW12 MX style mechanical keyboard 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, SW13 MX style mechanical keyboard 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, SW14 MX style mechanical keyboard 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, SW15 MX style mechanical keyboard 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, SW16 MX style mechanical keyboard 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, SW17 MX style mechanical keyboard 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, SW18 MX style mechanical keyboard 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, SW19 MX style mechanical keyboard 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, SW2 MX style mechanical keyboard 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, SW20 MX style mechanical keyboard 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, SW21 MX style mechanical keyboard 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, SW22 MX style mechanical keyboard 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, SW23 MX style mechanical keyboard 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, SW24 MX style mechanical keyboard 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, SW25 MX style mechanical keyboard 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, SW26 MX style mechanical keyboard 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, SW27 MX style mechanical keyboard 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, SW28 MX style mechanical keyboard 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, SW29 MX style mechanical keyboard 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, SW3 MX style mechanical keyboard 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, SW30 MX style mechanical keyboard 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, SW31 MX style mechanical keyboard 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, SW32 MX style mechanical keyboard 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, SW33 MX style mechanical keyboard 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, SW34 MX style mechanical keyboard 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, SW35 MX style mechanical keyboard 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, SW36 MX style mechanical keyboard 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, SW37 MX style mechanical keyboard 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, SW38 MX style mechanical keyboard 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, SW39 MX style mechanical keyboard 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, SW4 MX style mechanical keyboard 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, SW40 MX style mechanical keyboard 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, SW41 MX style mechanical keyboard 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, SW42 MX style mechanical keyboard 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, SW43 MX style mechanical keyboard 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, SW44 MX style mechanical keyboard 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, SW45 MX style mechanical keyboard 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, SW46 MX style mechanical keyboard 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, SW47 MX style mechanical keyboard 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, SW48 MX style mechanical keyboard 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, SW49 MX style mechanical keyboard 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, SW5 MX style mechanical keyboard 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, SW50 MX style mechanical keyboard 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, SW51 MX style mechanical keyboard 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, SW52 MX style mechanical keyboard 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, SW53 MX style mechanical keyboard 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, SW54 MX style mechanical keyboard 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, SW55 MX style mechanical keyboard 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, SW56 MX style mechanical keyboard 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, SW57 MX style mechanical keyboard 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, SW58 MX style mechanical keyboard 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, SW59 MX style mechanical keyboard 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, SW6 MX style mechanical keyboard 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, SW60 MX style mechanical keyboard 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, SW61 MX style mechanical keyboard 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, SW62 MX style mechanical keyboard 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, SW63 MX style mechanical keyboard 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, SW64 MX style mechanical keyboard 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, SW65 MX style mechanical keyboard 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, SW66 MX style mechanical keyboard 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, SW67 MX style mechanical keyboard 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, SW68 MX style mechanical keyboard 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, SW69 MX style mechanical keyboard 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, SW7 MX style mechanical keyboard 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, SW70 MX style mechanical keyboard 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, SW71 MX style mechanical keyboard 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, SW72 MX style mechanical keyboard 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, SW73 MX style mechanical keyboard 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, SW74 MX style mechanical keyboard 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, SW75 MX style mechanical keyboard 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, SW76 MX style mechanical keyboard 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, SW77 MX style mechanical keyboard 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, SW78 MX style mechanical keyboard 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, SW79 SSAL220100, SW8 MX style mechanical keyboard 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, SW80 K2-1187SQ-A4SW-06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

Commit message: Logos, extra pins, routing
- Loki65 logo added
- Gondolindrim logo added
- Extra remaining pins added
- Finish routing
- DRC pending
Parts:
- removed X2: USB pins, acheron_Connectors:PinHeader_1x4_P2.54mm_Vertical, symbol Connector_Generic:Conn_01x04
- added C26, C27, C28, C29, C30, C31, C32, C33, C34, C35, C36, C37, C38, C39, C40, C41, C42, C43: 100n, Capacitor_SMD:C_0805_2012Metric, symbol Device:C
- added D79, D80, D81, D82, D83, D84, D85, D86, D87, D88, D89, D90, D91, D92, D93, D94, D95, D96: WS2812B-2020, acheron_Components:LED_WS2812_2020, symbol acheron_Symbols:WS2812B-2020
- added GR1: Gondo Logo, gondolindrim_kicad_logos:gondolindrim_circuit-tree_10.4x12, symbol Mechanical:MountingHole
- added GR2: Loki Helmet Logo, loki65_lib:loki-helmet_18x10mm_plated, symbol Mechanical:MountingHole
- added J1: EXTRA_PINS, acheron_Connectors:PinHeader_1x9_P2.54mm_Vertical, symbol Connector_Generic:Conn_01x09
- added LED1, LED2: LED, acheron_Components:LED_THT_2.54mm, symbol acheron_Symbols:LED
- added R23, R24, R25, R26, R27, R28, R29, R30, R31, R32, R33, R34, R35, R36, R37, R38, R39, R40: 3R, Resistor_SMD:R_0805_2012Metric, symbol Device:R_Small
- added R3: 10k, Resistor_SMD:R_0805_2012Metric, symbol Device:R_Small
- added R6: 1k, Resistor_SMD:R_0805_2012Metric, symbol Device:R_Small
- renumbered C23 to C16, C24 to C17, C25 to C18, C16 to C19, C17 to C20, C18 to C21, C19 to C22, C20 to C23, C21 to C24, C22 to C25, D77 to D70, D78 to D71, D70 to D72, D71 to D73, D72 to D74, D73 to D75, D74 to D76, D75 to D77, D76 to D78, J1 to J2, R15 to R10, R17 to R11, R18 to R12, R19 to R13, R20 to R14, R16 to R15, R8 to R16, R9 to R17, R10 to R18, R11 to R19, R12 to R20, R13 to R21, R14 to R22, R3 to R4, R4 to R5, R5 to R7, R6 to R8, R7 to R9
Connections:
- net C15 is gone; now on net C14: SW15.1, SW31.1, SW46.1, SW63.1, SW73.1
- net 3V3: now also J1.1 (Pin_1)
- net 5V: now also LED1.A, LED2.A, R23.2, R24.2, R25.2, R26.2, R27.2, R28.2, R29.2, R30.2, R31.2, R32.2, R33.2, R34.2, R35.2, R36.2, R37.2, R38.2, R39.2, R40.2
- net C10: now also SW11.1, SW27.1, SW42.1, SW59.1, SW69.1, U2.45 (PB8); no longer SW10.1, SW26.1, SW41.1, SW58.1
- net C11: now also SW12.1, SW28.1, SW43.1, SW60.1, SW70.1, SW78.1, U2.46 (PB9); no longer SW11.1, SW27.1, SW42.1, SW59.1, SW69.1
- net C12: now also SW13.1, SW29.1, SW44.1, SW61.1, SW71.2, U2.2 (PC13); no longer SW12.1, SW28.1, SW43.1, SW60.1, SW70.1, SW78.1
- net C13: now also SW14.1, SW16.1, SW30.1, SW45.1, SW48.1, SW62.1, SW72.1, U2.3 (PC14_OSC32IN); no longer SW13.1, SW29.1, SW44.1, SW61.1, SW71.1
- net C14: now also U2.4 (PC15_OSC32OUT); no longer SW14.1, SW16.1, SW30.1, SW45.1, SW48.1, SW62.1, SW72.1
- net C5: now also U2.38 (PA15)
- net C6: now also U2.10 (PA0-WKUP)
- net C8: now also SW25.2, SW40.1, SW57.1, SW9.2, U2.40 (PB4); no longer SW24.2, SW39.1, SW56.1, SW8.1
- net C9: now also SW10.1, SW26.1, SW41.1, SW58.1, U2.41 (PB5); no longer SW25.2, SW40.1, SW57.1, SW9.2
- net CAPS_INDICATOR: now also U2.12 (PA2), R6.2; no longer U2.19 (PB1)
- net GND: now also C26.2, C27.2, C28.2, C29.2, C30.2, C31.2, C32.2, C33.2, C34.2, C35.2, C36.2, C37.2, C38.2, C39.2, C40.2, C41.2, C42.2, C43.2, D79.2 (VSS), D80.2 (VSS), D81.2 (VSS), D82.2 (VSS), D83.2 (VSS), D84.2 (VSS), D85.2 (VSS), D86.2 (VSS), D87.2 (VSS), D88.2 (VSS), D89.2 (VSS), D90.2 (VSS), D91.2 (VSS), D92.2 (VSS), D93.2 (VSS), D94.2 (VSS), D95.2 (VSS), D96.2 (VSS), J1.9 (Pin_9), R3.1
- net PB2/BOOT1: now also R3.2
- net R4: now also U2.11 (PA1); no longer U2.10 (PA0-WKUP)
- net RGB_5V: now also D71.3 (DIN); no longer D73.3 (DIN)
- net at D78.1 (DOUT): now also D79.3 (DIN); no longer D72.3 (DIN)
- net PA3: now reaches U2.13 (PA3)
- net PA3: now also J1.2 (Pin_2)
- net PA4: now reaches U2.14 (PA4)
- net PA4: now also J1.3 (Pin_3)
- net PA5: now reaches U2.15 (PA5)
- net PA5: now also J1.4 (Pin_4)
- net PA7: now reaches U2.17 (PA7)
- net PA7: now also J1.6 (Pin_6)
- net PB0: now reaches U2.18 (PB0)
- net PB0: now also J1.7 (Pin_7)
- net C7: now reaches U2.39 (PB3)
- net C7: now also SW24.2, SW39.1, SW56.1, SW8.1
- net at D71.1 (DOUT): now also D72.3 (DIN)
- net at D67.2 (A): now also SW71.1; no longer SW71.2
- net at D72.1 (DOUT): now also D73.3 (DIN)
- net LED_PWM renamed PA6
- net PA6: now also J1.5 (Pin_5)
- new net: D92.1 (DOUT), D93.3 (DIN)
- new net: D91.1 (DOUT), D92.3 (DIN)
- new net: C39.1, D92.4 (VDD), R36.1
- new net: C29.1, D82.4 (VDD), R26.1
- new net: C34.1, D87.4 (VDD), R31.1
- new net: C33.1, D86.4 (VDD), R30.1
- new net: C37.1, D90.4 (VDD), R34.1
- new net: D94.1 (DOUT), D95.3 (DIN)
- new net: D93.1 (DOUT), D94.3 (DIN)
- new net: C41.1, D94.4 (VDD), R38.1
- new net: C31.1, D84.4 (VDD), R28.1
- new net: C30.1, D83.4 (VDD), R27.1
- new net: C32.1, D85.4 (VDD), R29.1
- new net: C27.1, D80.4 (VDD), R24.1
- new net: C26.1, D79.4 (VDD), R23.1
- new net: C42.1, D95.4 (VDD), R39.1
- new net: D87.1 (DOUT), D88.3 (DIN)
- new net: D86.1 (DOUT), D87.3 (DIN)
- new net: D80.1 (DOUT), D81.3 (DIN)
- new net: D79.1 (DOUT), D80.3 (DIN)
- new net: D84.1 (DOUT), D85.3 (DIN)
- new net: D83.1 (DOUT), D84.3 (DIN)
- new net: C36.1, D89.4 (VDD), R33.1
- new net: D95.1 (DOUT), D96.3 (DIN)
- new net: D90.1 (DOUT), D91.3 (DIN)
- new net: C38.1, D91.4 (VDD), R35.1
- new net: C40.1, D93.4 (VDD), R37.1
- new net: D82.1 (DOUT), D83.3 (DIN)
- new net: D81.1 (DOUT), D82.3 (DIN)
- new net: D85.1 (DOUT), D86.3 (DIN)
- new net: D89.1 (DOUT), D90.3 (DIN)
- new net: C43.1, D96.4 (VDD), R40.1
- new net: LED1.K, LED2.K, R6.1
- new net: C28.1, D81.4 (VDD), R25.1
- new net: C35.1, D88.4 (VDD), R32.1
- new net: D88.1 (DOUT), D89.3 (DIN)
- new net PB1: J1.8 (Pin_8), U2.19 (PB1)
Other:
- note added: "SWITCH MATRIX"
- moved on the sheet: C13, C14, C15, C16, C17, C18, C19, C20, C21, C22, C23, C24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

Commit message: Add label, run DRC, expose B13
- Label for revision Alpha-rc1 added
- Gondolindrim and Loki65 logos had soldermask clearance added to 0.5mm
- DRC ran and errors corrected
- Pin B13 exposed
Parts:
- added GR3: Lok65 label, loki65_lib:loki65_label, symbol Mechanical:MountingHole
- J1: footprint acheron_Connectors:PinHeader_1x9_P2.54mm_Vertical -> acheron_Connectors:PinHeader_1x10_P2.54mm_Vertical; symbol Connector_Generic:Conn_01x09 -> Connector_Generic:Conn_01x10; now in the parts list
- renumbered C14 to C1, C7 to C10, C16 to C11, C17 to C12, C8 to C13, C9 to C14, C10 to C15, C11 to C16, C12 to C17, C15 to C2, C1 to C3, C2 to C4, C3 to C5, C4 to C6, C5 to C7, C13 to C8, C6 to C9, D70 to D1, D9 to D10, D10 to D11, D11 to D12, D12 to D13, D13 to D14, D14 to D15, D15 to D16, D16 to D17, D17 to D18, D18 to D19, D1 to D2, D19 to D20, D20 to D21, D21 to D22, D22 to D23, D23 to D24, D24 to D25, D25 to D26, D26 to D27, D27 to D28, D28 to D29, D2 to D3, D29 to D30, D30 to D31, D31 to D32, D32 to D33, D33 to D34, D34 to D35, D35 to D36, D36 to D37, D37 to D38, D38 to D39, D3 to D4, D39 to D40, D40 to D41, D41 to D42, D42 to D43, D43 to D44, D44 to D45, D45 to D46, D46 to D47, D47 to D48, D48 to D49, D4 to D5, D49 to D50, D50 to D51, D51 to D52, D52 to D53, D53 to D54, D54 to D55, D55 to D56, D56 to D57, D57 to D58, D58 to D59, D5 to D6, D59 to D60, D60 to D61, D61 to D62, D62 to D63, D63 to D64, D64 to D65, D65 to D66, D66 to D67, D67 to D68, D68 to D69, D6 to D7, D69 to D70, D7 to D8, D8 to D9, R11 to R10, R12 to R11, R6 to R12, R10 to R3, R3 to R4, R7 to R5, R8 to R6, R4 to R7, R9 to R8, R5 to R9, SW79 to SW1, SW8 to SW10, SW9 to SW11, SW10 to SW12, SW11 to SW13, SW12 to SW14, SW13 to SW15, SW14 to SW16, SW15 to SW17, SW16 to SW18, SW17 to SW19, SW80 to SW2, SW18 to SW20, SW19 to SW21, SW20 to SW22, SW21 to SW23, SW22 to SW24, SW23 to SW25, SW24 to SW26, SW25 to SW27, SW26 to SW28, SW27 to SW29, SW1 to SW3, SW28 to SW30, SW29 to SW31, SW30 to SW32, SW31 to SW33, SW32 to SW34, SW33 to SW35, SW34 to SW36, SW35 to SW37, SW36 to SW38, SW37 to SW39, SW2 to SW4, SW38 to SW40, SW39 to SW41, SW40 to SW42, SW41 to SW43, SW42 to SW44, SW43 to SW45, SW44 to SW46, SW45 to SW47, SW46 to SW48, SW47 to SW49, SW3 to SW5, SW48 to SW50, SW49 to SW51, SW50 to SW52, SW51 to SW53, SW52 to SW54, SW53 to SW55, SW54 to SW56, SW55 to SW57, SW56 to SW58, SW57 to SW59, SW4 to SW6, SW58 to SW60, SW59 to SW61, SW60 to SW62, SW61 to SW63, SW62 to SW64, SW63 to SW65, SW64 to SW66, SW65 to SW67, SW66 to SW68, SW67 to SW69, SW5 to SW7, SW68 to SW70, SW69 to SW71, SW70 to SW72, SW71 to SW73, SW72 to SW74, SW73 to SW75, SW74 to SW76, SW75 to SW77, SW76 to SW78, SW77 to SW79, SW6 to SW8, SW78 to SW80, SW7 to SW9, U3 to U1, U1 to U2, U2 to U3
Connections:
- net GND: now also J1.10 (Pin_10); no longer J1.9 (Pin_9)
- net PA3: now also J1.3 (Pin_3); no longer J1.2 (Pin_2)
- net PA4: now also J1.4 (Pin_4); no longer J1.3 (Pin_3)
- net PA5: now also J1.5 (Pin_5); no longer J1.4 (Pin_4)
- net PA6: now also J1.6 (Pin_6); no longer J1.5 (Pin_5)
- net PA7: now also J1.7 (Pin_7); no longer J1.6 (Pin_6)
- net PB0: now also J1.8 (Pin_8); no longer J1.7 (Pin_7)
- net PB1: now also J1.9 (Pin_9); no longer J1.8 (Pin_8)
- net PB13: now reaches U3.26 (PB13)
- net PB13: now also J1.2 (Pin_2)
- no-connect marks 3 -> 2

Commit message: Remove double BOOT1 resistor, add metadata
- Removed a double resistor grounding BOOT1
- Edited component metadata
- Release-ready
Parts:
- removed R6: 10k, Resistor_SMD:R_0805_2012Metric, symbol Device:R_Small
- C11, C12: Specification Tantallum 10V -> Tantallum 10V or more
- C13, C14, C16: Specification (none) -> MLCC 10V or more
- D10, D11, D12, D13, D14, D15, D16, D17, D18, D19, D2, D20, D21, D22, D23, D24, D25, D26, D27, D28, D29, D3, D30, D31, D32, D33, D34, D35, D36, D37, D38, D39, D4, D40, D41, D42, D43, D44, D45, D46, D47, D48, D49, D5, D50, D51, D52, D53, D54, D55, D56, D57, D58, D59, D6, D60, D61, D62, D63, D64, D65, D66, D67, D68, D69, D7, D70, D8, D9: Specification (none) -> Small-signal switching diode
- D71, D72, D73, D74, D75, D76, D77, D78, D79, D80, D81, D82, D83, D84, D85, D86, D87, D88, D89, D90, D91, D92, D93, D94, D95, D96: value WS2812B-2020 -> WS2812C-2020; Manufacturer (none) -> Worldsemi; Manufacturer Part Number (none) -> WS2812C-2020; Package (none) -> 2020; Specification (none) -> Serial addressable integrated controller RGB LEDs 2020 pack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; Vendor Part Number (none) -> LCSC C965556
- J1: renamed from J2; Specification (none) -> 16-pin USB type C 2.0 female connector
- U2: Specification (none) -> 256kB (32kBx8) I2C EEPROM
- U3: Manufacturer Part Number STM32F411 -> STM32F411CEU6; Specification (none) -> Cortex-M4+ 512kB flash microcontroller UFQFPN package
- X2: renamed from J1; now left out of the parts list
- Y1: Specification (none) -> 8MHz 3225-4P oscillator crystal
- renumbered R11 to R10, R12 to R11, R13 to R12, R14 to R13, R15 to R14, R16 to R15, R17 to R16, R18 to R17, R19 to R18, R20 to R19, R21 to R20, R22 to R21, R23 to R22, R24 to R23, R25 to R24, R26 to R25, R27 to R26, R28 to R27, R29 to R28, R30 to R29, R31 to R30, R32 to R31, R33 to R32, R34 to R33, R35 to R34, R36 to R35, R37 to R36, R38 to R37, R39 to R38, R40 to R39, R5 to R4, R4 to R5, R7 to R6, R8 to R7, R9 to R8, R10 to R9
Other:
- note added: "GRAPHICS"
- moved on the sheet: GR1, GR2, GR3, R5
